Commit message: Initial commit

File: src/mobile_robot_sim/urdf/DeliveryRobot_2.urdf (robot description, URDF)
Before this commit: robot DeliveryRobot_2, 11 links, 10 joints
Links:
- link FL_Wheel: geometry collision sphere radius=0.06; visual mesh filename=file:///home/zeinazz/design_ws/install/mobile_robot_sim/sha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
- link FR_Wheel: geometry collision sphere radius=0.06; visual mesh filename=file:///home/zeinazz/design_ws/install/mobile_robot_sim/sha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
- link Lid: geometry collision box size=0.39 0.47 0.02; visual mesh filename=file:///home/zeinazz/design_ws/install/mobile_robot_sim/sha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
- link RL_Wheel: geometry collision sphere radius=0.06; visual mesh filename=file:///home/zeinazz/design_ws/install/mobile_robot_sim/sha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
- link RR_Wheel: geometry collision sphere radius=0.06; visual mesh filename=file:///home/zeinazz/design_ws/install/mobile_robot_sim/sha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
- link RobotBody: geometry collision box size=0.39 0.47 0.14; visual mesh filename=file:///home/zeinazz/design_ws/install/mobile_robot_sim/sha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
- link ultrasonic_back_link: geometry collision cylinder length=0.005 radius=0.005; visual cylinder length=0.005 radius=0.005
- link ultrasonic_front_link: geometry collision cylinder length=0.005 radius=0.005; visual cylinder length=0.005 radius=0.005
- link ultrasonic_left_link: geometry collision cylinder length=0.005 radius=0.005; visual cylinder length=0.005 radius=0.005
- link ultrasonic_right_link: geometry collision cylinder length=0.005 radius=0.005; visual cylinder length=0.005 radius=0.005
Joints:
- joint FL_Joint: limit effort=2 velocity=2 -> effort=2 velocity=20
- joint FR_Joint: axis 0 0 1 -> 0 0 -1; limit effort=2 velocity=2 -> effort=2 velocity=20
- joint Lid_Joint: limit lower=0 upper=0.18 effort=2 velocity=2 -> lower=0 upper=0.18 effort=100 velocity=2
- joint RL_Joint: limit effort=2 velocity=2 -> effort=2 velocity=20
- joint RR_Joint: axis 0 0 1 -> 0 0 -1; limit effort=2 velocity=2 -> effort=2 velocity=20
- joint ultrasonic_back_joint: origin xyz=-0.20 0.0 0.07 rpy=0 0 3.14159 -> xyz=-0.25 0.0 0.07 rpy=0 0 3.14159
- joint ultrasonic_front_joint: origin xyz=0.20 0.0 0.07 rpy=0 0 0 -> xyz=0.25 0.0 0.07 rpy=0 0 0
- joint ultrasonic_left_joint: origin xyz=0.0 -0.24 0.07 rpy=0 0 1.5708 -> xyz=0.0 -0.24 0.07 rpy=0 0 -1.5708
- joint ultrasonic_right_joint: origin xyz=0.0 0.24 0.07 rpy=0 0 -1.5708 -> xyz=0.0 0.24 0.07 rpy=0 0 1.5708

Commit message: First_Static_Obstacle

File: src/mobile_robot_sim/urdf/DeliveryRobot_2.urdf (robot description, URDF)
Before this commit: robot DeliveryRobot_2, 11 links, 10 joints
Links:
- link FL_Wheel: geometry collision sphere radius=0.06; visual mesh filename=package://mobile_robot_sim/meshes/FL_Wheel.STL
- link FR_Wheel: geometry collision sphere radius=0.06; visual mesh filename=package://mobile_robot_sim/meshes/FR_Wheel.STL
- link Lid: geometry collision box size=0.39 0.47 0.02; visual mesh filename=package://mobile_robot_sim/meshes/Lid.STL
- link RL_Wheel: geometry collision sphere radius=0.06; visual mesh filename=package://mobile_robot_sim/meshes/RL_Wheel.STL
- link RR_Wheel: geometry collision sphere radius=0.06; visual mesh filename=package://mobile_robot_sim/meshes/RR_Wheel.STL
- link RobotBody: geometry collision box size=0.39 0.47 0.14; visual mesh filename=package://mobile_robot_sim/meshes/RobotBody.STL
Joints:
- joint Lid_Joint: limit lower=0 upper=0.18 effort=100 velocity=2 -> lower=0 upper=0.14 effort=100 velocity=2
