Commit message: First_Target

File: install/mobile_robot_sim/share/mobile_robot_sim/urdf/DeliveryRobot_2.urdf (robot description, URDF)
Before this commit: robot DeliveryRobot_2, 11 links, 10 joints
Joints:
- joint FL_Joint: limit effort=2 velocity=20 -> effort=20 velocity=20
- joint FR_Joint: limit effort=2 velocity=20 -> effort=20 velocity=20
- joint RL_Joint: limit effort=2 velocity=20 -> effort=20 velocity=20
- joint RR_Joint: limit effort=2 velocity=20 -> effort=20 velocity=20
